File: Phobri64/_autosave-Phobri64.kicad_sch (KiCad schematic)
At the start: 76 parts, among them J1 Stick_To_Mobo, J2 USB_B_Mini, J3 Conn_02x05_Counter_Clockwise, J4 Conn_01x01, J5 L_Board, J6 R_Board, J7 N64_Intf, J8 Mobo_To_Stick, J9 HoriStyleStick, SW1 A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

Commit message: Review notes
Other:
- note added: "(X) Shield resistor to both pins?"
- note removed: "Shield resistor to both pins?"
Changed lines of the file:
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@@
     (effects (font (size 2.54 2.54)) (justify left bottom))
   )
-  (text "Shield resistor to both pins?" (at 190.5 228.6 0)
+  (text "(X) Shield resistor to both pins?" (at 190.5 228.6 0)
     (effects (font (size 2 2) (color 255 0 0 1)) (justify left bottom))
   )
