File: Phobri64/_autosave-Phobri64.kicad_pcb (KiCad board)
At the start: 2 copper layers, 99.5 x 65.7 mm, 156 parts, among them J12 Mobo_To_Stick, J2 HoriStyleStick, J3 Conn_01x03, J4 L_Board, J5 R_Board, J6 N64_Intf, J7 Stick_To_Mobo, J8 USB_C_Receptacle, J9 Conn_01x03, SW1 A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

Commit message: b silkscreen additions
Parts:
- T_SW_3: value S -> Start
Other:
- board text added: "1V1"
- board text added: "3V3"
- board text added: "3V3 TX RX CTS RTS GND"
- board text added: "A"
- board text added: "B"
- board text added: "CD"
- board text added: "CL"
- board text added: "CR"
- board text added: "CU"
- board text added: "DD"
- board text added: "DL"
- board text added: "DR"
- board text added: "DU"
- board text added: "L"
- board text added: "N"
- board text added: "P"
- board text added: "Start"
- board text added: "ZL"
